Commit message: Rotated kuka coupler frame in order to avoid rpy singularities

File: soft_hand_klampt_description/meshes/accesories/kuka_coupler_floating.urdf.xacro (robot description, xacro)
@@ -24,5 +24,5 @@
   </link>
   <joint name="${parent}_${name}_base_joint" type="fixed">
-    <origin xyz="0 0 0.023" rpy="0 0 0"/>
+    <origin xyz="0 0 0.023" rpy="0 0 0.7854"/>
     <parent link="${name}_bottom"/>
     <child link="${name}"/>
